File: Assembly KICad/Assembly KICad.kicad_pcb (KiCad board)
At the start: 2 copper layers, 66 parts, among them J1 AudioJack2_Ground, J2 Conn_01x03_Pin, J3 CVOUT, J4 PDOUT, J5 AudioJack3, J6 AudioJack3, Q1 Q_NPN_BCE, Q2 Q_NPN_BCE, Q3 Q_NPN_BCE, Q4 Q_NPN_BCE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

Commit message: Kicad schematics & Pics
Parts:
- removed AudioOUT1: AudioJack2_Ground, Package_DIP:DIP-14_W7.62mm
- removed J1: AudioJack2_Ground, Connector_Audio:Jack_6.35mm_Neutrik_NJ3FD-V_Vertical
- J3, J4: footprint Connector_PinSocket_2.54mm:PinSocket_1x01_P2.54mm_Horizontal -> Connector_PinSocket_2.54mm:PinSocket_1x01_P2.54mm_Vertical
- RV1, RV2, RV3, RV4, RV5: footprint Potentiometer_THT:Potentiometer_Bourns_3386P_Vertical -> Potentiometer_THT:Potentiometer_Bourns_3386W_Horizontal
- U2: footprint Package_DIP:DIP-8_W7.62mm_Socket_LongPads -> Package_DIP:DIP-8_W7.62mm
- moved J2 159.9 mm to (196.5, 148.6)
- moved RV1 65.5 mm to (82.7, 36.4)
- moved Q4 60.3 mm to (103.5, 53.6)
- moved Q1 60.3 mm to (103.5, 36.2)
- moved Q2 60.3 mm to (103.5, 42.0)
- moved Q3 60.3 mm to (103.5, 47.8)
- moved RV2 56.5 mm to (82.7, 43.1)
- moved RV3 49.2 mm to (82.7, 49.7)
- moved D1 46.7 mm to (92.4, 34.8)
- moved D2 46.7 mm to (92.4, 38.3)
- moved D3 46.7 mm to (92.4, 41.9)
- moved D4 46.7 mm to (92.4, 45.4)
- moved D5 46.7 mm to (92.4, 49.0)
- moved D6 46.7 mm to (92.4, 52.5)
- moved D7 46.7 mm to (92.4, 56.1)
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
Commit message: Adding schematics on Kicad as well as adding some details
-updated schematics
-updated footprints
-updated 3D models
Parts:
- removed J6: AudioJack3, Connector_Audio:Jack_6.35mm_Neutrik_NJ3FD-V_Vertical
- added D12: LED, LED_THT:LED_D3.0mm_Horizontal_O1.27mm_Z2.0mm, F.Cu at (59.7, 63.7)
- added J1: AudioJack2, Connector_Audio:Jack_6.35mm_Neutrik_NJ2FD-V_Vertical, F.Cu at (106.7, 25.9)
- added R34: 4.7K, Resistor_THT:R_Axial_DIN0204_L3.6mm_D1.6mm_P7.62mm_Horizontal, F.Cu at (54.4, 59.5)
- J2: footprint Connector_Phoenix_MC_HighVoltage:PhoenixContact_MC_1,5_3-G-5.08_1x03_P5.08mm_Horizontal -> Connector_Phoenix_MC_HighVoltage:PhoenixContact_MCV_1,5_3-G-5.08_1x03_P5.08mm_Vertical
- J3, J4: footprint Connector_PinSocket_2.54mm:PinSocket_1x01_P2.54mm_Vertical -> Connector_PinHeader_2.54mm:PinHeader_1x01_P2.54mm_Vertical
- J5: value AudioJack3 -> AudioJack2; footprint Connector_Audio:Jack_6.35mm_Neutrik_NJ3FD-V_Vertical -> Connector_Audio:Jack_6.35mm_Neutrik_NJ2FD-V_Vertical
- RV1, RV2, RV3, RV4, RV5: footprint Potentiometer_THT:Potentiometer_Bourns_3386W_Horizontal -> Potentiometer_THT:Potentiometer_Bourns_3386P_Vertical
- moved J2 106.6 mm to (113.1, 82.1)
- moved RV5 96.6 mm to (179.3, 61.0)
- moved RV4 85.6 mm to (168.2, 61.0)
- moved RV3 75.3 mm to (157.1, 61.0)
- moved RV2 65.8 mm to (146.0, 61.0)
- moved RV1 57.7 mm to (135.0, 61.0)
- moved J5 36.0 mm to (123.2, 25.9)
- moved D8 20.0 mm to (68.5, 62.6)
- moved R13 20.0 mm to (78.8, 24.6)
- moved R14 20.0 mm to (78.8, 27.8)
- moved R15 20.0 mm to (78.8, 30.9)
- moved R16 20.0 mm to (78.8, 34.1)
- moved R17 20.0 mm to (78.8, 37.2)
- moved R18 20.0 mm to (78.8, 40.4)
- moved R19 20.0 mm to (78.8, 43.5)
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