File: Schematics in KiCad/Assembly KICad/Assembly KICad.kicad_sch (KiCad schematic)
At the start: 66 parts, among them J1 AudioJack2, J2 Conn_01x03_Pin, J3 CVOUT, J4 PDOUT, J5 AudioJack2, Q1 Q_NPN_BCE, Q2 Q_NPN_BCE, Q3 Q_NPN_BCE, Q4 Q_NPN_BCE, SW1 SW_DPDT_x2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

Commit message: Power analysis & Updating The Rapport
full power analysis
full schematics on kicad
PICS for each block
small adjustments in the schematics
Parts:
- added J10: -12Vss, Connector_PinHeader_2.54mm:PinHeader_1x01_P2.54mm_Vertical, symbol Connector:Conn_01x01_Socket
- added J11: -12ss, Connector_PinHeader_2.54mm:PinHeader_1x01_P2.54mm_Vertical, symbol Connector:Conn_01x01_Socket
- added J6: CVOUT, Connector_PinHeader_2.54mm:PinHeader_1x01_P2.54mm_Vertical, symbol Connector:Conn_01x01_Socket
- added J7: PDOUT, Connector_PinHeader_2.54mm:PinHeader_1x01_P2.54mm_Vertical, symbol Connector:Conn_01x01_Socket
- added J8: AMPOUT, Connector_PinHeader_2.54mm:PinHeader_1x01_P2.54mm_Vertical, symbol Connector:Conn_01x01_Socket
- added J9: AMPOUT/OUT, Connector_PinHeader_2.54mm:PinHeader_1x01_P2.54mm_Vertical, symbol Connector:Conn_01x01_Socket
- J3: value CVOUT -> CVOUT(AMPIN)
- J4: value PDOUT -> PDOUT(IN)
- R30, R31, R32, R33: value 50K -> 4.7K
Connections:
- net +12: now also Q2.3 (E), R31.1; no longer U3.8 (V+)
- net -12: no longer U3.4 (V-)
- net CVOUT: now also J6.1 (Pin_1)
- net PDOUT: now also J7.1 (Pin_1)
- net at RV5.2, RV5.3, U3.1: now also J8.1 (Pin_1); no longer R19.2
- new net: J11.1 (Pin_1), U3.4 (V-)
- new net: J10.1 (Pin_1), U3.8 (V+)
- new net: J9.1 (Pin_1), R19.2
Other:
- note added: "Optional Blocks"
- moved on the sheet: D10, D11, D12, D8, D9, J2, J3, J4, Q1, Q2, Q3, Q4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

Commit message: Starting The PCB Layout
Parts:
- J1: value AudioJack2 -> AudioIn
- J5: value AudioJack2 -> AudioOut
Connections:
- net +12: no longer Q1.2 (C), Q2.2 (C), Q2.3 (E), Q3.2 (C), Q4.2 (C), R31.1
- net at J10.1 (Pin_1), U3.8 (V+): now also Q1.2 (C), Q2.2 (C), Q2.3 (E), Q3.2 (C), Q4.2 (C), R31.1
Changed lines of the file:
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@@
 	)
 	(junction
+		(at 187.96 57.15)
+		(diameter 0)
+		(color 0 0 0 0)
+	)
+	(junction
 		(at 256.54 88.9)
 		(diameter 0)
@@
 	(wire
 		(pts
-			(xy 237.49 49.53) (xy 246.38 49.53)
-		)
-		(stroke
-			(width 0)
-			(type default)
-		)
-	)
-	(wire
-		(pts
 			(xy 262.89 74.93) (xy 264.16 74.93)
 		)
@@
 	(wire
 		(pts
+			(xy 187.96 49.53) (xy 187.96 57.15)
+		)
+		(stroke
+			(width 0)
+			(type default)
+		)
+	)
+	(wire
+		(pts
 			(xy 59.69 15.24) (xy 59.69 19.05)
 		)
@@
 	(wire
 		(pts
+			(xy 187.96 49.53) (xy 246.38 49.53)
+		)
+		(stroke
+			(width 0)
+			(type default)
+		)
+	)
+	(wire
+		(pts
 			(xy 45.72 27.94) (xy 48.26 27.94)
 		)
@@
 		)
 	)
-	(global_label "+12"
-		(shape input)
-		(at 237.49 49.53 180)
-		(fields_autoplaced yes)
-		(effects
-			(font
-				(size 1.27 1.27)
-			)
-			(justify right)
-		)
-		(property "Intersheetrefs" "${INTERSHEET_REFS}"
-			(at 230.5134 49.53 0)
-			(effects
-				(font
-					(size 1.27 1.27)
-				)
-				(justify right)
-				(hide yes)
-			)
-		)
-	)
 	(global_label "COMPOUT"
 		(shape input)
@@
 			)
 		)
-		(property "Value" "AudioJack2"
+		(property "Value" "AudioOut"
 			(at 92.075 175.26 0)
 			(effects
@@
 			)
 		)
-		(property "Value" "AudioJack2"
+		(property "Value" "AudioIn"
 			(at 34.925 125.73 0)
 			(effects
