File: Schematics in KiCad/Assembly KICad/Assembly KICad.kicad_pcb (KiCad board)
At the start: 2 copper layers, 66 parts, among them J1 AudioJack2, J2 Conn_01x03_Pin, J3 CVOUT, J4 PDOUT, J5 AudioJack2, Q1 Q_NPN_BCE, Q2 Q_NPN_BCE, Q3 Q_NPN_BCE, Q4 Q_NPN_BCE, SW1 SW_DPDT_x2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

Commit message: Power analysis & Updating The Rapport
full power analysis
full schematics on kicad
PICS for each block
small adjustments in the schematics
Parts:
- added J6: CVOUT, Connector_PinHeader_2.54mm:PinHeader_1x01_P2.54mm_Vertical, F.Cu at (140.0, 28.5)
- added J7: PDOUT, Connector_PinHeader_2.54mm:PinHeader_1x01_P2.54mm_Vertical, F.Cu at (145.0, 28.5)
- added J8: AMPOUT, Connector_PinHeader_2.54mm:PinHeader_1x01_P2.54mm_Vertical, F.Cu at (100.0, 75.4)
- added J9: AMPOUT/OUT, Connector_PinHeader_2.54mm:PinHeader_1x01_P2.54mm_Vertical, F.Cu at (100.0, 80.0)
- J3: value CVOUT -> CVOUT(AMPIN)
- J4: value PDOUT -> PDOUT(IN)
Connections:
- R19 pad 2: Net-(R19-Pad2) -> Net-(J9-Pin_1)
- RV5 pad 2: Net-(R19-Pad2) -> Net-(J8-Pin_1)
- RV5 pad 3: Net-(R19-Pad2) -> Net-(J8-Pin_1)
- U3 pad 1: Net-(R19-Pad2) -> Net-(J8-Pin_1)

Commit message: Starting The PCB Layout
Parts:
- added J10: -12Vss, Connector_PinHeader_2.54mm:PinHeader_1x01_P2.54mm_Vertical, F.Cu at (59.1, 156.5)
- added J11: -12ss, Connector_PinHeader_2.54mm:PinHeader_1x01_P2.54mm_Vertical, F.Cu at (59.1, 161.1)
- J1: value AudioJack2 -> AudioIn
- J5: value AudioJack2 -> AudioOut
- R30, R31, R32, R33: value 50K -> 4.7K
- moved R19 207.6 mm to (263.4, 138.5)
- moved D12 203.2 mm to (262.5, 49.5)
- moved SW1 191.4 mm to (261.5, 152.5)
- moved R34 190.0 mm to (244.2, 51.5)
- moved R11 179.5 mm to (242.9, 97.5)
- moved R12 179.5 mm to (242.9, 100.7)
- moved J9 165.9 mm to (254.5, 140.5)
- moved R8 162.0 mm to (222.4, 96.5)
- moved D1 157.2 mm to (259.7, 93.3)
- moved D2 157.2 mm to (259.7, 96.8)
- moved D3 157.2 mm to (259.7, 100.4)
- moved D4 157.2 mm to (259.7, 104.0)
- moved D5 157.2 mm to (259.7, 107.5)
- moved D6 157.2 mm to (259.7, 111.0)
- moved D7 157.2 mm to (259.7, 114.6)
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Connections:
- Q2 pad 3: Net-(Q2-E) -> +12
- R31 pad 1: Net-(Q2-E) -> +12
- U3 pad 4: -12 -> Net-(J11-Pin_1)
- U3 pad 8: +12 -> Net-(J10-Pin_1)
Other:
- board outline added: 125 x 133 mm

Commit message: Starting the pcb layout and routing process
Parts:
- added REF**: MountingHole_3.2mm_M3, MountingHole:MountingHole_3.2mm_M3, F.Cu at (-245.8, -76.0)
- added REF**: MountingHole_3.2mm_M3, MountingHole:MountingHole_3.2mm_M3, F.Cu at (-227.8, -88.0)
- added REF**: MountingHole_3.2mm_M3, MountingHole:MountingHole_3.2mm_M3, F.Cu at (-245.8, -88.0)
- added REF**: MountingHole_3.2mm_M3, MountingHole:MountingHole_3.2mm_M3, F.Cu at (-227.8, -76.0)
- J1, J2, J5: moved to B.Cu
- moved D8 327.6 mm to (-277.4, 42.3)
- moved D10 327.6 mm to (-265.4, 42.3)
- moved D11 327.6 mm to (-259.4, 42.3)
- moved D9 327.6 mm to (-271.4, 42.3)
- moved J4 322.2 mm to (-195.3, 45.5)
- moved J8 313.8 mm to (-189.4, 80.3)
- moved RV1 312.8 mm to (-66.0, 10.1)
- moved RV2 308.5 mm to (-50.4, 10.1)
- moved U2 308.5 mm to (-41.2, 50.6)
- moved RV3 304.7 mm to (-35.5, 10.1)
- moved RV4 297.3 mm to (-16.8, 10.0)
- moved R23 287.9 mm to (-252.3, 91.4)
- moved R25 287.9 mm to (-173.5, 108.9)
- moved Q2 283.9 mm to (-221.5, 82.3)
- moved J10 281.9 mm to (-202.9, 52.5)
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Connections:
- Q1 pad 2: +12 -> Net-(J10-Pin_1)
- Q2 pad 2: +12 -> Net-(J10-Pin_1)
- Q2 pad 3: +12 -> Net-(J10-Pin_1)
- Q3 pad 2: +12 -> Net-(J10-Pin_1)
- Q4 pad 2: +12 -> Net-(J10-Pin_1)
- R31 pad 1: +12 -> Net-(J10-Pin_1)
Routing:
- net Net-(U1D-+): track 0.00 -> 24.9 mm
- net +12: track 0.00 -> 20.9 mm
- net Net-(U1B--): track 0.00 -> 17.4 mm
- net CVO+: track 0.00 -> 12.2 mm
- net CVO-: track 0.00 -> 9.41 mm
- net Net-(R1-Pad2): track 0.00 -> 4.32 mm
- net Net-(U1D--): track 0.00 -> 2.54 mm
- added copper zone on B.Cu, net GND
Other:
- board size 125 x 133 mm -> 70 x 100 mm

Commit message: Updates
Parts:
- removed REF** (x4): MountingHole_3.2mm_M3, MountingHole:MountingHole_3.2mm_M3
- D10, D11, D12, D8, D9, Q1, Q2, Q3, Q4, R25, R26, R27, R28, R30, R31, R32, R33, RV1, RV2, RV3, RV4, RV5: moved to B.Cu
- J2: moved to F.Cu
- moved D8 505.3 mm to (220.2, 130.5), turned to 180 degrees
- moved D9 492.7 mm to (213.3, 130.5), turned to 180 degrees
- moved D10 480.0 mm to (206.4, 130.5), turned to 180 degrees
- moved D11 467.3 mm to (199.6, 130.5), turned to 180 degrees
- moved R23 460.2 mm to (203.6, 28.4)
- moved R30 453.2 mm to (217.5, 119.8), turned to -90 degrees
- moved Q2 448.8 mm to (225.3, 124.5), turned to 180 degrees
- moved R31 446.9 mm to (211.7, 119.8), turned to -90 degrees
- moved R32 439.9 mm to (205.2, 119.8), turned to -90 degrees
- moved R33 431.3 mm to (197.0, 119.8), turned to -90 degrees
- moved J11 425.0 mm to (221.9, 45.0), turned to 90 degrees
- moved R29 417.1 mm to (195.5, 80.1), turned to 90 degrees
- moved J4 415.5 mm to (219.7, 26.3), turned to 90 degrees
- moved J10 410.9 mm to (207.0, 23.8), turned to 90 degrees
- moved Q1 409.5 mm to (216.1, 113.3), turned to -90 degrees
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Routing:
- net Net-(J10-Pin_1): track 0.00 -> 158.0 mm
- net -12: track 0.00 -> 94.2 mm
- net +12: track 20.9 -> 114.8 mm
- net COMPOUT: track 0.00 -> 56.2 mm
- net CVOUT: track 0.00 -> 53.2 mm
- net Net-(U2A-+): track 0.00 -> 51.9 mm
- net Net-(R24-Pad2): track 0.00 -> 51.4 mm
- net Net-(SW1A-B): track 0.00 -> 43.7 mm
- net Net-(Q1-B): track 0.00 -> 41.7 mm
- net Net-(U1D-+): track 24.9 -> 64.4 mm
- net PDOUT: track 0.00 -> 39.0 mm
- net Net-(D3-K): track 0.00 -> 35.2 mm
- net CVO-: track 9.41 -> 44.2 mm
- net GND: track 0.00 -> 31.7 mm
- net Net-(R16-Pad2): track 0.00 -> 27.9 mm
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Other:
- board size 70 x 100 mm -> 80 x 120 mm
- board text added: "Amplification"
- board text added: "Attack"
- board text added: "AudioIN"
- board text added: "AudioOut"
- board text added: "IND"
- board text added: "Ratio"
- board text added: "Release"
- board text added: "Threshold"

Commit message: Updating Rapport
Other:
- board text added: "By Saif Abdessayed https://github.com/GarablueX"
Changed lines of the file:
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@@
+		)
+	)
+	(gr_text "By Saif Abdessayed\nhttps://github.com/GarablueX"
+		(at 249.61 24.12 0)
+		(layer "B.SilkS")
+		(effects
+			(font
+				(size 1 1)
+				(thickness 0.1)
+			)
+			(justify left bottom mirror)
 		)
 	)
