File: Schematics in KiCad/Assembly KICad/Assembly without optional blocks/Assembly without optional blocks.kicad_pcb (KiCad board)
At the start: 2 copper layers, 84.9 x 65.8 mm, 39 parts, among them J1 AudioIn, J2 Conn_01x03_Pin, J5 AudioOut, U1 TL074, U2 TL072

Commit message: adding the first layouts and 3d views
Parts:
- added REF**: MountingHole_2.2mm_M2, MountingHole:MountingHole_2.2mm_M2, F.Cu at (159.3, 33.2)
- added REF**: MountingHole_2.2mm_M2, MountingHole:MountingHole_2.2mm_M2, F.Cu at (159.3, 94.1)
- added REF**: MountingHole_2.2mm_M2, MountingHole:MountingHole_2.2mm_M2, F.Cu at (80.4, 33.2)
- added REF**: MountingHole_2.2mm_M2, MountingHole:MountingHole_2.2mm_M2, F.Cu at (80.4, 94.1)
- added T-12: TestPoint_Pad_1.0x1.0mm, TestPoint:TestPoint_Pad_1.0x1.0mm, F.Cu at (95.7, 94.1)
- added T12: TestPoint_Pad_1.0x1.0mm, TestPoint:TestPoint_Pad_1.0x1.0mm, F.Cu at (96.9, 85.4)
- added TCOMPOUT: TestPoint_Pad_1.0x1.0mm, TestPoint:TestPoint_Pad_1.0x1.0mm, B.Cu at (129.1, 36.1)
- added TCVOUT: TestPoint_Pad_1.0x1.0mm, TestPoint:TestPoint_Pad_1.0x1.0mm, F.Cu at (137.9, 61.8)
- moved R5 128.5 mm to (142.6, 31.8)
- moved D2 120.4 mm to (158.5, 43.0)
- moved D12 120.4 mm to (86.0, 81.9)
- moved D7 120.4 mm to (115.9, 57.1)
- moved J1 120.4 mm to (124.9, 80.9)
- moved R15 120.4 mm to (103.4, 59.9)
- moved R2 120.4 mm to (115.0, 36.0)
- moved R34 120.4 mm to (97.2, 82.1)
- moved C1 120.4 mm to (124.6, 58.7)
- moved C2 120.4 mm to (142.6, 65.7)
- moved D1 120.4 mm to (150.9, 38.4)
- moved D3 120.4 mm to (150.9, 47.6)
- moved D5 120.4 mm to (150.9, 64.0)
- moved J5 120.4 mm to (147.9, 80.9)
- moved R1 120.4 mm to (120.8, 46.8)
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Routing:
- net CVO+: track 42.6 -> 34.3 mm
- net Net-(D1-A): track 4.44 -> 11.1 mm
- net CVOUT: track 56.0 -> 60.7 mm
- net COMPOUT: track 81.9 -> 86.1 mm
- net +12: track 123.5 -> 127.0 mm
- net -12: track 112.1 -> 114.4 mm
- net Net-(J1-PadT): track 44.1 -> 45.1 mm
Other:
- board size 84.9 x 65.8 mm -> 84.9 x 66.9 mm
- board text added: "+12"
- board text added: "-12"
- board text added: "Aduio in"
- board text added: "Attack"
- board text added: "Audio Out"
- board text added: "By Saif Abdessayed"
- board text added: "GND"
- board text added: "IND LED"
- board text added: "Ratio"
- board text added: "Release"
- board text added: "Threshold"
- board text added: "https://github.com/GarablueX"
